File: keyboard.kicad_pcb (KiCad board)
At the start: 2 copper layers, 285 x 94.6 mm, 245 parts, among them IC1 ATMEGA32U4, P1 CONN_3X2, Q1 2N7002, Q2 Q_PMOS_GDS, SW1 JUMPER, SW2 CONN_3, U1 TP4056, U2 MDBT40, U3 IS31FL3733, X1 ASX3F

Commit message: Fix Bugs
Parts:
- removed C14: 104, Resistor_SMD:R_0603_1608Metric
- removed P1: CONN_3X2, random-keyboard-parts:Jumper-UserFriendly
- removed R11: 10k, Resistor_SMD:R_0603_1608Metric
- R12: value 10k -> 20k
- moved R12 1.06 mm to (171.6, 153.2)
- renumbered CHG to D1, Done to D2
Connections:
- U3 pad 49: GND -> (no net)
Routing:
- net /DFU: track 34.5 -> 1.83 mm
- net Net-(C11-Pad2): track 44.1 -> 17.2 mm
- net /FACRST: track 19.1 -> 2.50 mm
- net /DIO_RST: track 17.8 -> 2.53 mm
- net /SWCLK: track 14.3 -> 2.50 mm
- net /BT_RX: track 77.2 -> 79.7 mm
- net Net-(U2-Pad28): track 0.00 -> 2.52 mm
- net Net-(U2-Pad26): track 0.00 -> 2.51 mm
- net Net-(R12-Pad1): track 7.90 -> 5.43 mm
- net /BT_TX: track 78.9 -> 81.2 mm
- net /leds/VCC_LED: track 164.4 -> 162.4 mm
- net /leds/CS13: track 330.7 -> 329.0 mm
- net VCC: track 138.8 -> 137.7 mm
- net GND: track 118.4 -> 118.8 mm, vias 401 -> 403
