File: keyboard.kicad_pcb (KiCad board)
At the start: 2 copper layers, 285 x 94.6 mm, 245 parts, among them IC1 ATMEGA32U4, P1 CONN_3X2, Q1 2N7002, Q2 Q_PMOS_GDS, SW1 JUMPER, SW2 CONN_3, U1 TP4056, U2 MDBT40, U3 IS31FL3733, X1 ASX3F

Commit message: 1st Gen BT-Keyboard
Parts:
- removed BAT1: CONN_2, Connector_PinHeader_2.54mm:PinHeader_1x02_P2.54mm_Vertical
- removed the C10 at (220.2, 125.6)
- removed C12, C13, C9: 1u, 0805:0805C
- removed C14, C15, C16, C17: 104, Resistor_SMD:R_0603_1608Metric
- removed CHG: CHG, 0805:0805D
- removed the D65 at (327.5, 98.2)
- removed Done: CHDONE, 0805:0805D
- removed Q1: 2N7002, Keebio-Parts:SOT-23_Handsoldering
- removed Q2: Q_PMOS_GDS, Keebio-Parts:SOT-23_Handsoldering
- removed R11, R12, R13, R14, R7, R8, R9: 10k, Resistor_SMD:R_0603_1608Metric
- removed the R6 at (103.7, 134.8)
- removed SW1: JUMPER, Button_Switch_SMD:SW_SPST_CK_RS282G05A3
- removed SW2: CONN_3, Button_Switch_THT:SW_Slide_1P2T_CK_OS102011MS2Q
- removed U1: TP4056, Keebio-Parts:SOIC-8_3.9x4.9mm_Pitch1.27mm
- removed U2: MDBT40, mdbt40_carrier:MDBT40_UART
- removed U3: IS31FL3733, Package_DFN_QFN:QFN-48-1EP_6x6mm_P0.4mm_EP4.2x4.2mm
- added BLUETOOTH: MDBT40, mdbt40_carrier:MDBT40_F, B.Cu at (216.6, 149.9)
- added C8: 1u, 0805:0805C, B.Cu at (82.9, 84.5)
- added D67: 1N4148, 0805:0805D, B.Cu at (341.6, 102.0)
- added DC1: LED, WS2812B:3528_LED, B.Cu at (63.8, 107.8)
- added JP1: JUMPER3, Jumper:SolderJumper-3_P1.3mm_Open_Pad1.0x1.5mm_NumberLabels, B.Cu at (231.1, 149.6)
- added JP2: JUMPER3, Jumper:SolderJumper-3_P1.3mm_Open_Pad1.0x1.5mm_NumberLabels, B.Cu at (233.6, 148.3)
- added LDO: 2N7002, Keebio-Parts:SOT-23_Handsoldering, B.Cu at (140.6, 147.4)
- added R4: 300, 0805:0805R, B.Cu at (68.9, 115.2)
- added REF**: Jumper-UserFriendly-Small, random-keyboard-parts:Jumper-UserFriendly-Small, B.Cu at (137.0, 144.8)
- added REF**: , tqfp:QFN_32U4, B.Cu at (161.2, 148.9)
- added RGB62: WS2812B, LED_SMD:LED_SK6812MINI_PLCC4_3.5x3.5mm_P1.75mm, B.Cu at (301.9, 131.1)
- added RGB63: WS2812B, LED_SMD:LED_SK6812MINI_PLCC4_3.5x3.5mm_P1.75mm, B.Cu at (257.3, 125.7)
- added RGB64: WS2812B, LED_SMD:LED_SK6812MINI_PLCC4_3.5x3.5mm_P1.75mm, B.Cu at (219.4, 125.8)
- added RGB65: WS2812B, LED_SMD:LED_SK6812MINI_PLCC4_3.5x3.5mm_P1.75mm, B.Cu at (181.6, 126.1)
- added RGB66: WS2812B, LED_SMD:LED_SK6812MINI_PLCC4_3.5x3.5mm_P1.75mm, B.Cu at (143.3, 125.9)
- added RGB67: WS2812B, LED_SMD:LED_SK6812MINI_PLCC4_3.5x3.5mm_P1.75mm, B.Cu at (101.0, 131.1)
- added RGB68: WS2812B, LED_SMD:LED_SK6812MINI_PLCC4_3.5x3.5mm_P1.75mm, B.Cu at (153.3, 106.5)
- added RGB69: WS2812B, LED_SMD:LED_SK6812MINI_PLCC4_3.5x3.5mm_P1.75mm, B.Cu at (134.0, 106.5)
- added RGB70: WS2812B, LED_SMD:LED_SK6812MINI_PLCC4_3.5x3.5mm_P1.75mm, B.Cu at (114.2, 106.8)
- added RGB71: WS2812B, LED_SMD:LED_SK6812MINI_PLCC4_3.5x3.5mm_P1.75mm, B.Cu at (68.2, 88.5)
- added RGB72: WS2812B, LED_SMD:LED_SK6812MINI_PLCC4_3.5x3.5mm_P1.75mm, B.Cu at (110.6, 88.8)
- added RGB73: WS2812B, LED_SMD:LED_SK6812MINI_PLCC4_3.5x3.5mm_P1.75mm, B.Cu at (147.3, 88.7)
- added RGB74: WS2812B, LED_SMD:LED_SK6812MINI_PLCC4_3.5x3.5mm_P1.75mm, B.Cu at (186.7, 89.1)
- added RGB75: WS2812B, LED_SMD:LED_SK6812MINI_PLCC4_3.5x3.5mm_P1.75mm, B.Cu at (224.3, 88.4)
- added RGB76: WS2812B, LED_SMD:LED_SK6812MINI_PLCC4_3.5x3.5mm_P1.75mm, B.Cu at (263.3, 88.9)
- added RGB77: WS2812B, LED_SMD:LED_SK6812MINI_PLCC4_3.5x3.5mm_P1.75mm, B.Cu at (301.0, 88.6)
- added RGB78: WS2812B, LED_SMD:LED_SK6812MINI_PLCC4_3.5x3.5mm_P1.75mm, B.Cu at (342.8, 75.5)
- added RGB81: WS2812B, WS2812B:WS2812-3528-with-sik, B.Cu at (335.8, 150.0)
- added S0: DTSM-6, dtsm:KSEM31GLFS, B.Cu at (91.4, 112.8)
- C1: renamed from C4; footprint Resistor_SMD:R_0603_1608Metric -> 0805:0805C
- C10: renamed from C11; value 104 -> 1u; footprint Resistor_SMD:R_0603_1608Metric -> 0805:0805C
- C2: renamed from C8; footprint Resistor_SMD:R_0603_1608Metric -> 0805:0805C
- C4: renamed from C2; footprint Resistor_SMD:R_0603_1608Metric -> 0805:0805C
- C5: renamed from C3; footprint Resistor_SMD:R_0603_1608Metric -> 0805:0805C
- C6: renamed from C5; footprint Resistor_SMD:R_0603_1608Metric -> 0805:0805C
- C7: renamed from C6; footprint Resistor_SMD:R_0603_1608Metric -> 0805:0805C
- IC1: footprint tqfp:QFN_32U4 -> tqfp:TQFP44
- R1: renamed from R2; footprint Resistor_SMD:R_0603_1608Metric -> 0805:0805R
- R10: value 10k -> 10K; footprint Resistor_SMD:R_0603_1608Metric -> 0805:0805R
- R2: renamed from R3; footprint Resistor_SMD:R_0603_1608Metric -> 0805:0805R
- R3: renamed from R5; footprint Resistor_SMD:R_0603_1608Metric -> 0805:0805R
- R5: renamed from R4; footprint Resistor_SMD:R_0603_1608Metric -> 0805:0805R
- R6: renamed from R1; footprint Resistor_SMD:R_0603_1608Metric -> 0805:0805R
- RGB1, RGB10, RGB11, RGB12, RGB13, RGB14, RGB15, RGB16, RGB17, RGB18, RGB19, RGB2, RGB20, RGB21, RGB22, RGB23, RGB24, RGB25, RGB26, RGB27, RGB28, RGB29, RGB3, RGB30, RGB31, RGB32, RGB33, RGB34, RGB35, RGB36, RGB37, RGB38, RGB39, RGB4, RGB40, RGB41, RGB42, RGB43, RGB44, RGB45, RGB46, RGB47, RGB48, RGB49, RGB5, RGB50, RGB51, RGB52, RGB53, RGB54, RGB55, RGB56, RGB57, RGB58, RGB59, RGB6, RGB60, RGB7, RGB8, RGB9: value LED_ARGB -> WS2812B; footprint WS2812B:RGB-3528-with-sik -> WS2812B:WS2812-3528-with-sik; moved to B.Cu
- RGB61: value LED_ARGB -> WS2812B; footprint WS2812B:RGB-3528-with-sik -> LED_SMD:LED_SK6812MINI_PLCC4_3.5x3.5mm_P1.75mm; moved to B.Cu
- moved R10 33.0 mm to (204.9, 148.1), turned to 0 degrees
- moved RGB61 19.5 mm to (339.0, 130.9), turned to 0 degrees
- moved D58 18.1 mm to (306.9, 113.5), turned to 270 degrees
- moved D10 17.9 mm to (108.1, 148.1), turned to 270 degrees
- moved D61 17.5 mm to (310.6, 73.2)
- moved D60 17.4 mm to (298.1, 148.1), turned to 270 degrees
- moved D26 17.2 mm to (176.5, 72.1)
- moved D18 17.2 mm to (153.2, 111.6), turned to 270 degrees
- moved D53 17.2 mm to (286.1, 110.5), turned to 270 degrees
- moved D36 17.1 mm to (214.3, 71.8)
- moved D56 17.1 mm to (290.7, 72.1)
- moved D51 17.1 mm to (271.7, 72.3)
- moved D65 17.0 mm to (321.2, 147.7), turned to 270 degrees
- moved D15 17.0 mm to (131.0, 148.2), turned to 270 degrees
- moved D5 17.0 mm to (83.3, 148.1), turned to 270 degrees
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- renumbered C7 to C3, D3 to CON, D4 to D1, D13 to D10, D14 to D11, D15 to D12, D16 to D13, D17 to D14, D18 to D15, D19 to D16, D20 to D17, D21 to D18, D22 to D19, D5 to D2, D23 to D21, D24 to D22, D25 to D23, D26 to D24, D27 to D26, D28 to D27, D29 to D28, D30 to D29, D6 to D3, D31 to D30, D32 to D31, D33 to D32, D34 to D33, D35 to D34, D7 to D4, D40 to D41, D41 to D42, D42 to D43, D43 to D44, D44 to D46, D45 to D47, D46 to D48, D47 to D49, D8 to D5, D49 to D51, D50 to D52, D51 to D53, D52 to D54, D53 to D55, D54 to D56, D55 to D57, D56 to D58, D57 to D59, D9 to D6, D58 to D60, D59 to D61, D60 to D62, D63 to D65, D64 to D66, D66 to D68, D67 to D69, D10 to D7, D68 to D70, D11 to D8, P1 to P2, S3 to S1, S13 to S10, S17 to S11, S18 to S12, S19 to S13, S20 to S14, S21 to S15, S22 to S16, S23 to S17, S24 to S18, S25 to S19, S4 to S2, S26 to S21, S27 to S22, S28 to S23, S29 to S24, S31 to S26, S32 to S27, S33 to S28, S34 to S29, S5 to S3, S37 to S311, S38 to S32, S39 to S33, S40 to S34, S41 to S36, S42 to S37, S43 to S38, S44 to S39, S6 to S4, S45 to S411, S46 to S42, S47 to S43, S48 to S44, S49 to S46, S50 to S47, S51 to S48, S52 to S49, S8 to S5, S55 to S51, S56 to S52, S57 to S53, S58 to S54, S59 to S55, S60 to S56, S61 to S57, S62 to S58, S63 to S59, S9 to S6, S64 to S60, S68 to S61, S69 to S62, S67 to S65, S77 to S66, S79 to S67, S80 to S68, S82 to S69, S10 to S7, S76 to S70, S11 to S8
Connections:
- C10 pad 2: Net-(C11-Pad2) -> VCC
- IC1 pad 10: /PWDN -> /MOSI
- IC1 pad 11: /BT_EN -> /MISO
- IC1 pad 18: /SCL -> /row1
- IC1 pad 19: /SDA -> /row2
- IC1 pad 20: /BT_TX -> /col8
- IC1 pad 21: /BT_RX -> /col14
- IC1 pad 38: /row2 -> /WS2812
- IC1 pad 39: /row1 -> Net-(IC1-Pad39)
- IC1 pad 7: VBUS -> VCC
- IC1 pad 8: /col14 -> /caps
- IC1 pad 9: /col8 -> /SCK
- P2 pad 1: Net-(C11-Pad2) -> VCC
- R10 pad 1: /SDA -> GND
- R10 pad 2: /leds/VCC_LED -> Net-(R10-Pad2)
- RGB1 pad 1: /leds/CS1 -> VCC
- RGB1 pad 2: /leds/SW3 -> Net-(RGB1-Pad2)
- RGB1 pad 3: /leds/SW2 -> GND
- RGB1 pad 4: /leds/SW1 -> /DIN_M
- RGB10 pad 1: /leds/CS10 -> VCC
- RGB10 pad 2: /leds/SW3 -> Net-(RGB10-Pad2)
- RGB10 pad 3: /leds/SW2 -> GND
- RGB10 pad 4: /leds/SW1 -> Net-(RGB10-Pad4)
- RGB11 pad 1: /leds/CS11 -> VCC
- RGB11 pad 2: /leds/SW3 -> Net-(RGB11-Pad2)
- RGB11 pad 3: /leds/SW2 -> GND
- RGB11 pad 4: /leds/SW1 -> Net-(RGB10-Pad2)
- RGB12 pad 1: /leds/CS12 -> VCC
- RGB12 pad 2: /leds/SW3 -> Net-(RGB12-Pad2)
- RGB12 pad 3: /leds/SW2 -> GND
- RGB12 pad 4: /leds/SW1 -> Net-(RGB11-Pad2)
- RGB13 pad 1: /leds/CS13 -> VCC
- RGB13 pad 2: /leds/SW3 -> Net-(RGB13-Pad2)
- RGB13 pad 3: /leds/SW2 -> GND
- RGB13 pad 4: /leds/SW1 -> Net-(RGB12-Pad2)
- RGB14 pad 1: /leds/CS14 -> VCC
- RGB14 pad 2: /leds/SW3 -> Net-(RGB14-Pad2)
- RGB14 pad 3: /leds/SW2 -> GND
- RGB14 pad 4: /leds/SW1 -> Net-(RGB13-Pad2)
- RGB15 pad 1: /leds/CS14 -> VCC
- RGB15 pad 2: /leds/SW6 -> Net-(RGB15-Pad2)
- RGB15 pad 3: /leds/SW5 -> GND
- RGB15 pad 4: /leds/SW4 -> Net-(RGB14-Pad2)
- RGB16 pad 1: /leds/CS13 -> VCC
- RGB16 pad 2: /leds/SW6 -> Net-(RGB16-Pad2)
- RGB16 pad 3: /leds/SW5 -> GND
- RGB16 pad 4: /leds/SW4 -> Net-(RGB15-Pad2)
- RGB17 pad 1: /leds/CS12 -> VCC
- RGB17 pad 2: /leds/SW6 -> Net-(RGB17-Pad2)
- RGB17 pad 3: /leds/SW5 -> GND
- RGB17 pad 4: /leds/SW4 -> Net-(RGB16-Pad2)
- RGB18 pad 1: /leds/CS11 -> VCC
- RGB18 pad 2: /leds/SW6 -> Net-(RGB18-Pad2)
- RGB18 pad 3: /leds/SW5 -> GND
- RGB18 pad 4: /leds/SW4 -> Net-(RGB17-Pad2)
- RGB19 pad 1: /leds/CS10 -> VCC
- RGB19 pad 2: /leds/SW6 -> Net-(RGB19-Pad2)
- RGB19 pad 3: /leds/SW5 -> GND
- RGB19 pad 4: /leds/SW4 -> Net-(RGB18-Pad2)
- RGB2 pad 1: /leds/CS2 -> VCC
- RGB2 pad 2: /leds/SW3 -> Net-(RGB2-Pad2)
- RGB2 pad 3: /leds/SW2 -> GND
- RGB2 pad 4: /leds/SW1 -> Net-(RGB1-Pad2)
- RGB20 pad 1: /leds/CS9 -> VCC
- RGB20 pad 2: /leds/SW6 -> Net-(RGB20-Pad2)
- RGB20 pad 3: /leds/SW5 -> GND
- RGB20 pad 4: /leds/SW4 -> Net-(RGB19-Pad2)
- RGB21 pad 1: /leds/CS8 -> VCC
- RGB21 pad 2: /leds/SW6 -> Net-(RGB21-Pad2)
- RGB21 pad 3: /leds/SW5 -> GND
- RGB21 pad 4: /leds/SW4 -> Net-(RGB20-Pad2)
- RGB22 pad 1: /leds/CS7 -> VCC
- RGB22 pad 2: /leds/SW6 -> Net-(RGB22-Pad2)
- RGB22 pad 3: /leds/SW5 -> GND
- RGB22 pad 4: /leds/SW4 -> Net-(RGB21-Pad2)
- RGB23 pad 1: /leds/CS6 -> VCC
- RGB23 pad 2: /leds/SW6 -> Net-(RGB23-Pad2)
- RGB23 pad 3: /leds/SW5 -> GND
- RGB23 pad 4: /leds/SW4 -> Net-(RGB22-Pad2)
- RGB24 pad 1: /leds/CS5 -> VCC
- RGB24 pad 2: /leds/SW6 -> Net-(RGB24-Pad2)
- RGB24 pad 3: /leds/SW5 -> GND
- RGB24 pad 4: /leds/SW4 -> Net-(RGB23-Pad2)
- RGB25 pad 1: /leds/CS4 -> VCC
- RGB25 pad 2: /leds/SW6 -> Net-(RGB25-Pad2)
- RGB25 pad 3: /leds/SW5 -> GND
- RGB25 pad 4: /leds/SW4 -> Net-(RGB24-Pad2)
- RGB26 pad 1: /leds/CS3 -> VCC
- RGB26 pad 2: /leds/SW6 -> Net-(RGB26-Pad2)
- RGB26 pad 3: /leds/SW5 -> GND
- RGB26 pad 4: /leds/SW4 -> Net-(RGB25-Pad2)
- RGB27 pad 1: /leds/CS2 -> VCC
- RGB27 pad 2: /leds/SW6 -> Net-(RGB27-Pad2)
- RGB27 pad 3: /leds/SW5 -> GND
- RGB27 pad 4: /leds/SW4 -> Net-(RGB26-Pad2)
- RGB28 pad 1: /leds/CS1 -> VCC
- RGB28 pad 2: /leds/SW6 -> Net-(RGB28-Pad2)
- RGB28 pad 3: /leds/SW5 -> GND
- RGB28 pad 4: /leds/SW4 -> Net-(RGB27-Pad2)
- RGB29 pad 1: /leds/CS1 -> VCC
- RGB29 pad 2: /leds/SW9 -> Net-(RGB29-Pad2)
- RGB29 pad 3: /leds/SW8 -> GND
- RGB29 pad 4: /leds/SW7 -> Net-(RGB28-Pad2)
- RGB3 pad 1: /leds/CS3 -> VCC
- RGB3 pad 2: /leds/SW3 -> Net-(RGB3-Pad2)
- RGB3 pad 3: /leds/SW2 -> GND
- RGB3 pad 4: /leds/SW1 -> Net-(RGB2-Pad2)
- RGB30 pad 1: /leds/CS2 -> VCC
- RGB30 pad 2: /leds/SW9 -> Net-(RGB30-Pad2)
- RGB30 pad 3: /leds/SW8 -> GND
- RGB30 pad 4: /leds/SW7 -> Net-(RGB29-Pad2)
- RGB31 pad 1: /leds/CS3 -> VCC
- RGB31 pad 2: /leds/SW9 -> Net-(RGB31-Pad2)
- RGB31 pad 3: /leds/SW8 -> GND
- RGB31 pad 4: /leds/SW7 -> Net-(RGB30-Pad2)
- RGB32 pad 1: /leds/CS4 -> VCC
- RGB32 pad 2: /leds/SW9 -> Net-(RGB32-Pad2)
- RGB32 pad 3: /leds/SW8 -> GND
- RGB32 pad 4: /leds/SW7 -> Net-(RGB31-Pad2)
- RGB33 pad 1: /leds/CS5 -> VCC
- RGB33 pad 2: /leds/SW9 -> Net-(RGB33-Pad2)
- RGB33 pad 3: /leds/SW8 -> GND
- RGB33 pad 4: /leds/SW7 -> Net-(RGB32-Pad2)
- RGB34 pad 1: /leds/CS6 -> VCC
- RGB34 pad 2: /leds/SW9 -> Net-(RGB34-Pad2)
- RGB34 pad 3: /leds/SW8 -> GND
- RGB34 pad 4: /leds/SW7 -> Net-(RGB33-Pad2)
- RGB35 pad 1: /leds/CS7 -> VCC
- RGB35 pad 2: /leds/SW9 -> Net-(RGB35-Pad2)
- RGB35 pad 3: /leds/SW8 -> GND
- RGB35 pad 4: /leds/SW7 -> Net-(RGB34-Pad2)
- RGB36 pad 1: /leds/CS8 -> VCC
- RGB36 pad 2: /leds/SW9 -> Net-(RGB36-Pad2)
- RGB36 pad 3: /leds/SW8 -> GND
- RGB36 pad 4: /leds/SW7 -> Net-(RGB35-Pad2)
- RGB37 pad 1: /leds/CS9 -> VCC
- RGB37 pad 2: /leds/SW9 -> Net-(RGB37-Pad2)
- RGB37 pad 3: /leds/SW8 -> GND
- RGB37 pad 4: /leds/SW7 -> Net-(RGB36-Pad2)
- RGB38 pad 1: /leds/CS10 -> VCC
- RGB38 pad 2: /leds/SW9 -> Net-(RGB38-Pad2)
- RGB38 pad 3: /leds/SW8 -> GND
- RGB38 pad 4: /leds/SW7 -> Net-(RGB37-Pad2)
- RGB39 pad 1: /leds/CS11 -> VCC
- RGB39 pad 2: /leds/SW9 -> Net-(RGB39-Pad2)
- RGB39 pad 3: /leds/SW8 -> GND
- RGB39 pad 4: /leds/SW7 -> Net-(RGB38-Pad2)
- RGB4 pad 1: /leds/CS4 -> VCC
- RGB4 pad 2: /leds/SW3 -> Net-(RGB4-Pad2)
- RGB4 pad 3: /leds/SW2 -> GND
- RGB4 pad 4: /leds/SW1 -> Net-(RGB3-Pad2)
- RGB40 pad 1: /leds/CS12 -> VCC
- RGB40 pad 2: /leds/SW9 -> Net-(RGB40-Pad2)
- RGB40 pad 3: /leds/SW8 -> GND
- RGB40 pad 4: /leds/SW7 -> Net-(RGB39-Pad2)
- RGB41 pad 1: /leds/CS13 -> VCC
- RGB41 pad 2: /leds/SW9 -> Net-(RGB41-Pad2)
- RGB41 pad 3: /leds/SW8 -> GND
- RGB41 pad 4: /leds/SW7 -> Net-(RGB40-Pad2)
- RGB42 pad 1: /leds/CS12 -> VCC
- RGB42 pad 2: /leds/SW12 -> Net-(RGB42-Pad2)
- RGB42 pad 3: /leds/SW11 -> GND
- RGB42 pad 4: /leds/SW10 -> Net-(RGB41-Pad2)
- RGB43 pad 1: /leds/CS11 -> VCC
- RGB43 pad 2: /leds/SW12 -> Net-(RGB43-Pad2)
- RGB43 pad 3: /leds/SW11 -> GND
- RGB43 pad 4: /leds/SW10 -> Net-(RGB42-Pad2)
- RGB44 pad 1: /leds/CS10 -> VCC
- RGB44 pad 2: /leds/SW12 -> Net-(RGB44-Pad2)
- RGB44 pad 3: /leds/SW11 -> GND
- RGB44 pad 4: /leds/SW10 -> Net-(RGB43-Pad2)
- RGB45 pad 1: /leds/CS9 -> VCC
- RGB45 pad 2: /leds/SW12 -> Net-(RGB45-Pad2)
- RGB45 pad 3: /leds/SW11 -> GND
- RGB45 pad 4: /leds/SW10 -> Net-(RGB44-Pad2)
- RGB46 pad 1: /leds/CS8 -> VCC
- RGB46 pad 2: /leds/SW12 -> Net-(RGB46-Pad2)
- RGB46 pad 3: /leds/SW11 -> GND
- RGB46 pad 4: /leds/SW10 -> Net-(RGB45-Pad2)
- RGB47 pad 1: /leds/CS7 -> VCC
- RGB47 pad 2: /leds/SW12 -> Net-(RGB47-Pad2)
- RGB47 pad 3: /leds/SW11 -> GND
- RGB47 pad 4: /leds/SW10 -> Net-(RGB46-Pad2)
- RGB48 pad 1: /leds/CS6 -> VCC
- RGB48 pad 2: /leds/SW12 -> Net-(RGB48-Pad2)
- RGB48 pad 3: /leds/SW11 -> GND
- RGB48 pad 4: /leds/SW10 -> Net-(RGB47-Pad2)
- RGB49 pad 1: /leds/CS5 -> VCC
- RGB49 pad 2: /leds/SW12 -> Net-(RGB49-Pad2)
- RGB49 pad 3: /leds/SW11 -> GND
- RGB49 pad 4: /leds/SW10 -> Net-(RGB48-Pad2)
- RGB5 pad 1: /leds/CS5 -> VCC
- RGB5 pad 2: /leds/SW3 -> Net-(RGB5-Pad2)
- RGB5 pad 3: /leds/SW2 -> GND
- RGB5 pad 4: /leds/SW1 -> Net-(RGB4-Pad2)
- RGB50 pad 1: /leds/CS4 -> VCC
- RGB50 pad 2: /leds/SW12 -> Net-(RGB50-Pad2)
- RGB50 pad 3: /leds/SW11 -> GND
- RGB50 pad 4: /leds/SW10 -> Net-(RGB49-Pad2)
- RGB51 pad 1: /leds/CS3 -> VCC
- RGB51 pad 2: /leds/SW12 -> Net-(RGB51-Pad2)
- RGB51 pad 3: /leds/SW11 -> GND
- RGB51 pad 4: /leds/SW10 -> Net-(RGB50-Pad2)
- RGB52 pad 1: /leds/CS2 -> VCC
- RGB52 pad 2: /leds/SW12 -> Net-(RGB52-Pad2)
- RGB52 pad 3: /leds/SW11 -> GND
- RGB52 pad 4: /leds/SW10 -> Net-(RGB51-Pad2)
- RGB53 pad 1: /leds/CS1 -> VCC
- RGB53 pad 2: /leds/SW12 -> Net-(RGB53-Pad2)
- RGB53 pad 3: /leds/SW11 -> GND
- RGB53 pad 4: /leds/SW10 -> Net-(RGB52-Pad2)
- RGB54 pad 1: /leds/CS16 -> VCC
- RGB54 pad 2: /leds/SW3 -> Net-(RGB54-Pad2)
- RGB54 pad 3: /leds/SW2 -> GND
- RGB54 pad 4: /leds/SW1 -> Net-(RGB53-Pad2)
- RGB55 pad 1: /leds/CS16 -> VCC
- RGB55 pad 2: /leds/SW6 -> Net-(RGB55-Pad2)
- RGB55 pad 3: /leds/SW5 -> GND
- RGB55 pad 4: /leds/SW4 -> Net-(RGB54-Pad2)
- RGB56 pad 1: /leds/CS16 -> VCC
- RGB56 pad 2: /leds/SW9 -> Net-(RGB56-Pad2)
- RGB56 pad 3: /leds/SW8 -> GND
- RGB56 pad 4: /leds/SW7 -> Net-(RGB55-Pad2)
- RGB57 pad 1: /leds/CS15 -> VCC
- RGB57 pad 2: /leds/SW9 -> Net-(RGB57-Pad2)
- RGB57 pad 3: /leds/SW8 -> GND
- RGB57 pad 4: /leds/SW7 -> Net-(RGB56-Pad2)
- RGB58 pad 1: /leds/CS16 -> VCC
- RGB58 pad 2: /leds/SW12 -> Net-(RGB58-Pad2)
- RGB58 pad 3: /leds/SW11 -> GND
- RGB58 pad 4: /leds/SW10 -> Net-(RGB57-Pad2)
- RGB59 pad 1: /leds/CS15 -> VCC
- RGB59 pad 2: /leds/SW12 -> Net-(RGB59-Pad2)
- RGB59 pad 3: /leds/SW11 -> GND
- RGB59 pad 4: /leds/SW10 -> Net-(RGB58-Pad2)
- RGB6 pad 1: /leds/CS6 -> VCC
- RGB6 pad 2: /leds/SW3 -> Net-(RGB6-Pad2)
- RGB6 pad 3: /leds/SW2 -> GND
- RGB6 pad 4: /leds/SW1 -> Net-(RGB5-Pad2)
- RGB60 pad 1: /leds/CS14 -> VCC
- RGB60 pad 2: /leds/SW12 -> Net-(RGB60-Pad2)
- RGB60 pad 3: /leds/SW11 -> GND
- RGB60 pad 4: /leds/SW10 -> Net-(RGB59-Pad2)
- RGB61 pad 1: /leds/CS13 -> VCC
- RGB61 pad 2: /leds/SW12 -> Net-(RGB61-Pad2)
- RGB61 pad 3: /leds/SW11 -> GND
- RGB61 pad 4: /leds/SW10 -> /DIN_D
- RGB7 pad 1: /leds/CS7 -> VCC
- RGB7 pad 2: /leds/SW3 -> Net-(RGB7-Pad2)
- RGB7 pad 3: /leds/SW2 -> GND
- RGB7 pad 4: /leds/SW1 -> Net-(RGB6-Pad2)
- RGB8 pad 1: /leds/CS8 -> VCC
- RGB8 pad 2: /leds/SW3 -> Net-(RGB8-Pad2)
- RGB8 pad 3: /leds/SW2 -> GND
- RGB8 pad 4: /leds/SW1 -> Net-(RGB7-Pad2)
- RGB9 pad 1: /leds/CS9 -> VCC
- RGB9 pad 2: /leds/SW3 -> Net-(RGB10-Pad4)
- RGB9 pad 3: /leds/SW2 -> GND
- RGB9 pad 4: /leds/SW1 -> Net-(RGB8-Pad2)
- USB1 pad 11: VBUS -> VCC
- USB1 pad 2: VBUS -> VCC
Routing:
- net VCC: track 138.8 -> 2068.4 mm, vias 9 -> 44
- net /leds/SW2: track 538.3 -> 0.00 mm, vias 18 -> 0
- net /leds/SW1: track 485.7 -> 0.00 mm, vias 18 -> 0
- net /leds/SW5: track 485.5 -> 0.00 mm, vias 20 -> 0
- net /leds/SW3: track 467.8 -> 0.00 mm, vias 18 -> 0
- net /leds/SW4: track 462.2 -> 0.00 mm, vias 18 -> 0
- net /leds/SW11: track 449.3 -> 0.00 mm, vias 16 -> 0
- net /leds/SW6: track 434.2 -> 0.00 mm, vias 22 -> 0
- net /leds/SW8: track 433.1 -> 0.00 mm, vias 15 -> 0
- net /leds/SW10: track 400.8 -> 0.00 mm, vias 18 -> 0
- net /leds/SW7: track 386.5 -> 0.00 mm, vias 17 -> 0
- net /leds/SW12: track 384.0 -> 0.00 mm, vias 18 -> 0
- net /leds/SW9: track 377.3 -> 0.00 mm, vias 16 -> 0
- net /leds/CS13: track 330.7 -> 0.00 mm, vias 8 -> 0
- net /leds/CS14: track 312.4 -> 0.00 mm, vias 8 -> 0
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- removed copper zone on B.Cu, net GND
- removed copper zone on F.Cu, net GND
- removed copper zone on F.Cu, net VBUS
Other:
- board text added: "Power Jump"
- board text removed: "V2.0"
