File: keyboard.sch (KiCad schematic (older format))
At the start: 36 parts, among them IC1 ATMEGA32U4, P1 CONN_3X2, Q1 2N7002, Q2 Q_PMOS_GDS, SW1 JUMPER, SW2 CONN_3, U1 TP4056, U2 MDBT40, X1 ASX3F

Commit message: default GH60 Keyboard
Parts:
- removed BAT1: CONN_2, Connector_PinHeader_2.54mm:PinHeader_1x02_P2.54mm_Vertical, symbol conn:CONN_2
- removed C10, C12, C13, C9: 1u, 0805:0805C, symbol device:C
- removed C11: 104, Resistor_SMD:R_0603_1608Metric, symbol device:C
- removed D1: CHG, 0805:0805D, symbol device:LED
- removed D2: CHDONE, 0805:0805D, symbol device:LED
- removed D3: LED, 0805:0805D, symbol device:LED
- removed JP1: Power, Keebio-Parts:solder_jumper, symbol device:JUMPER
- removed P1: CONN_3X2, random-keyboard-parts:Jumper-UserFriendly, symbol conn:CONN_3X2
- removed Q1: 2N7002, Keebio-Parts:SOT-23_Handsoldering, symbol Transistor_FET:2N7002
- removed Q2: Q_PMOS_GDS, Keebio-Parts:SOT-23_Handsoldering, symbol Device:Q_PMOS_GDS
- removed R1: 5.1K, Resistor_SMD:R_0603_1608Metric, symbol device:R
- removed R6: 1k, Resistor_SMD:R_0603_1608Metric, symbol device:R
- removed R7, R8: 10k, Resistor_SMD:R_0603_1608Metric, symbol device:R
- removed SW1: JUMPER, Button_Switch_SMD:SW_SPST_CK_RS282G05A3, symbol device:JUMPER
- removed SW2: CONN_3, Button_Switch_THT:SW_Slide_1P2T_CK_OS102011MS2Q, symbol conn:CONN_3
- removed U1: TP4056, Keebio-Parts:SOIC-8_3.9x4.9mm_Pitch1.27mm, symbol XLED:TP4056
- removed U2: MDBT40, mdbt40_carrier:MDBT40_UART, symbol keyboard-rescue:MDBT40-mdbt40
- removed USB1: HRO-TYPE-C-31-M-12, Type-C:HRO-TYPE-C-31-M-12-HandSoldering, symbol keyboard-rescue:HRO-TYPE-C-31-M-12-Type-C
- added DF10, DF11, DF20, DF201, DF3, DW1, DW2, DW3, DW4: LED, mx1a:MX1A-led_no3d, symbol LED
- added DF21, DF211, DF22, DF221, DF23, DF231, DF232: LED, symbol LED
- added J1: MINI, usb:67503, symbol USBMINI_B05
- added P1, P10, P11, P12, P13, P14, P15, P16, P17, P18, P19, P2, P20, P21, P22, P23, P24, P25, P26, P27, P28, P29, P3, P30, P31, P32, P33, P34, P35, P36, P37, P38, P39, P4, P40, P41, P42, P5, P6, P7, P8, P9: CONN_1, symbol CONN_1
- added R10, R11, R12, R13, R14, R15, R6, R7, R8, R9: R, symbol R
- added S0: DTSM-6, dtsm:KSEM31GLFS, symbol DTSM-6
- C1: renamed from C4; footprint Resistor_SMD:R_0603_1608Metric -> 0805:0805C; symbol device:C -> C
- C2: renamed from C8; footprint Resistor_SMD:R_0603_1608Metric -> 0805:0805C; symbol device:C -> C
- C3: renamed from C7; symbol device:C -> C
- C4: renamed from C2; footprint Resistor_SMD:R_0603_1608Metric -> 0805:0805C; symbol device:C -> C
- C5: renamed from C3; footprint Resistor_SMD:R_0603_1608Metric -> 0805:0805C; symbol device:C -> C
- C6: renamed from C5; footprint Resistor_SMD:R_0603_1608Metric -> 0805:0805C; symbol device:C -> C
- C7: renamed from C6; footprint Resistor_SMD:R_0603_1608Metric -> 0805:0805C; symbol device:C -> C
- C8: renamed from C1; symbol device:C -> C
- IC1: footprint tqfp:QFN_32U4 -> tqfp:TQFP44; symbol atmega32u4:ATMEGA32U4 -> ATMEGA32U4
- R1: renamed from R2; footprint Resistor_SMD:R_0603_1608Metric -> 0805:0805R; symbol device:R -> R
- R2: renamed from R3; footprint Resistor_SMD:R_0603_1608Metric -> 0805:0805R; symbol device:R -> R
- R3: renamed from R5; footprint Resistor_SMD:R_0603_1608Metric -> 0805:0805R; symbol device:R -> R
- R5: renamed from R4; footprint Resistor_SMD:R_0603_1608Metric -> 0805:0805R; symbol device:R -> R
- X1: symbol aker:ASX4 -> ASX4
Connections:
- net labels added: GPIO0, GPIO1, GPIO2, GPIO3, MISO, MOSI, SCK, caps, ~RES~
- net labels removed: BAT_V, BT_EN, BT_RX, BT_TX, CONed, D+, D-, DFU, DIO_RST, FACRST, PWDN, SCL, SDA, SWCLK, VBUS
- wire segments 242 -> 205
- no-connect marks 29 -> 5
Other:
- note added: "Backlight expansion\nconnector (top)"
- note added: "Universal expansion\nconnector (bottom)"
