File: leds.sch (KiCad schematic (older format))
At the start: 72 parts, among them U3 IS31FL3733

Commit message: Fix Bugs
Parts:
- removed C14: 104, Resistor_SMD:R_0603_1608Metric, symbol device:C
- removed R11: 10k, Resistor_SMD:R_0603_1608Metric, symbol device:R
- R12: value 10k -> 20k
Changed lines of the file:
@@
-	1    0    0    -1
-$EndComp
-$Comp
-L device:C C?
-U 1 1 6253FDCE
-P 11950 12950
-AR Path="/6253FDCE" Ref="C?"  Part="1"
-AR Path="/5DD60643/6253FDCE" Ref="C14"  Part="1"
-F 0 "C14" H 12085 12996 50  0000 L CNN
-F 1 "104" H 12085 12905 50  0000 L CNN
-F 2 "Resistor_SMD:R_0603_1608Metric" H 11950 12950 60  0001 C CNN
-F 3 "" H 11950 12950 60  0001 C CNN
-	1    11950 12950
 	1    0    0    -1
 $EndComp
@@
 Wire Wire Line
 	8750 12150 8750 12300
-$Comp
-L device:R R?
-U 1 1 62D37705
-P 11600 12500
-AR Path="/62D37705" Ref="R?"  Part="1"
-AR Path="/5DD60643/62D37705" Ref="R11"  Part="1"
-F 0 "R11" V 11680 12500 50  0000 C CNN
-F 1 "10k" V 11600 12500 50  0000 C CNN
-F 2 "Resistor_SMD:R_0603_1608Metric" H 11600 12500 60  0001 C CNN
-F 3 "http://www.tme.eu/pl/Document/e5152f6c2c4f933b61676f6de7ae79a8/dcrcw.pdf" H 11600 12500 60  0001 C CNN
-F 4 "Vishay" H 11600 12500 60  0001 C CNN "Vendor"
-F 5 "CRCW080510K0JNTABC" H 11600 12500 60  0001 C CNN "Product"
-F 6 "TME" H 11600 12500 60  0001 C CNN "Supplier"
-F 7 "CRCW080510K0JNTABC" H 11600 12500 60  0001 C CNN "Supplier Symbol"
-	1    11600 12500
-	1    0    0    -1
-$EndComp
 $Comp
 L device:R R?
@@
 AR Path="/5DD60643/62DA9C2F" Ref="R12"  Part="1"
 F 0 "R12" V 11680 13000 50  0000 C CNN
-F 1 "10k" V 11600 13000 50  0000 C CNN
+F 1 "20k" V 11600 13000 50  0000 C CNN
 F 2 "Resistor_SMD:R_0603_1608Metric" H 11600 13000 60  0001 C CNN
 F 3 "http://www.tme.eu/pl/Document/e5152f6c2c4f933b61676f6de7ae79a8/dcrcw.pdf" H 11600 13000 60  0001 C CNN
@@
 Wire Wire Line
 	10200 12750 11600 12750
-Connection ~ 11600 12750
 Wire Wire Line
 	10300 14200 11600 14200
@@
 	11600 14200 11600 13900
 Connection ~ 10300 14200
-Wire Wire Line
-	11600 12250 11600 12200
-Wire Wire Line
-	11600 12200 11100 12200
 Connection ~ 9850 12200
 Wire Wire Line
@@
 NoConn ~ 9550 12300
 NoConn ~ 9050 12300
-Wire Wire Line
-	11600 12750 11950 12750
-Wire Wire Line
-	11950 13250 11600 13250
-Wire Wire Line
-	11950 13150 11950 13250
 Connection ~ 11600 13250
 $Comp
@@
 	1    0    0    -1
 $EndComp
-Connection ~ 11600 12200
-Wire Wire Line
-	11950 13250 12500 13250
 Wire Wire Line
 	13300 13250 13300 13150
-Connection ~ 11950 13250
 Wire Wire Line
 	12900 13150 12900 13250
@@
 Wire Wire Line
 	12900 12750 12900 12200
-Wire Wire Line
-	11600 12200 12900 12200
 Wire Wire Line
 	8750 12150 9150 12150
@@
 Wire Wire Line
 	2600 3800 4600 3800
+Wire Wire Line
+	11100 12200 12900 12200
+Wire Wire Line
+	11600 13250 12500 13250
 $EndSCHEMATC
