File: leds.sch (KiCad schematic (older format))
At the start: 72 parts, among them U3 IS31FL3733

Commit message: default GH60 Keyboard
Parts:
- removed C14, C15, C16, C17: 104, Resistor_SMD:R_0603_1608Metric, symbol device:C
- removed R10, R11, R12, R13, R14, R9: 10k, Resistor_SMD:R_0603_1608Metric, symbol device:R
- removed RGB1, RGB10, RGB11, RGB12, RGB13, RGB14, RGB15, RGB16, RGB17, RGB18, RGB19, RGB2, RGB20, RGB21, RGB22, RGB23, RGB24, RGB25, RGB26, RGB27, RGB28, RGB29, RGB3, RGB30, RGB31, RGB32, RGB33, RGB34, RGB35, RGB36, RGB37, RGB38, RGB39, RGB4, RGB40, RGB41, RGB42, RGB43, RGB44, RGB45, RGB46, RGB47, RGB48, RGB49, RGB5, RGB50, RGB51, RGB52, RGB53, RGB54, RGB55, RGB56, RGB57, RGB58, RGB59, RGB6, RGB60, RGB61, RGB7, RGB8, RGB9: LED_ARGB, WS2812B:RGB-3528-with-sik, symbol Device:LED_ARGB
- removed U3: IS31FL3733, Package_DFN_QFN:QFN-48-1EP_6x6mm_P0.4mm_EP4.2x4.2mm, symbol XLED:IS31FL3733
- added DB02, DB04, DB041, DB06, DB07, DB09, DB11, DB14, DB16, DB17, DB19, DB21, DB22, DB23, DB24, DB26, DB27, DB28, DB29, DB30, DB301, DB302, DB31, DB32, DB33, DB34, DB36, DB37, DB38, DB39, DB41, DB42, DB43, DB44, DB46, DB47, DB48, DB49, DB50, DB51, DB52, DB53, DB54, DB56, DB57, DB58, DB59, DB61, DB62, DB63, DB66, DB661, DB67, DB68, DB681, DB682, DB69: LED, mx1a:MX1A-led_no3d, symbol LED
- added DB05, DB051, DB10, DB101, DB102, DB15, DB151, DB55, DB551: LED, symbol LED
Connections:
- net labels added: lcol1, lcol10, lcol11, lcol12, lcol13, lcol14, lcol2, lcol3, lcol4, lcol5, lcol6, lcol7, lcol8, lcol9, lrow1, lrow2, lrow3, lrow4, lrow5
- net labels removed: CS1, CS10, CS11, CS12, CS13, CS14, CS15, CS16, CS2, CS3, CS4, CS5, CS6, CS7, CS8, CS9, GND, I2CRST, SCL, SDA, SDB, SW1, SW10, SW11, SW12, SW2, SW3, SW4, SW5, SW6, SW7, SW8, SW9, VCC_LED
- wire segments 655 -> 74
- no-connect marks 4 -> 0
Other:
- note added: "Fn"
- note added: "caps\nlock"
- note added: "esc"
- note added: "led on extra key\nafter backspace"
- note added: "only rightmost position\nleft and center are\nhandled by the controller"
- note added: "wasd\ncluster"
- note removed: "'"
- note removed: ","
- note removed: "-"
- note removed: "."
- note removed: "/"
- note removed: "0"
- note removed: "1"
- note removed: "2"
- note removed: "3"
- note removed: "4\n"
- note removed: "5"
- note removed: "6"
- note removed: "7"
- note removed: "8"
- note removed: "9"
- note removed: ";"
- note removed: "="
- note removed: "A"
- note removed: "B"
- note removed: "C"
- note removed: "CAPSLOCK"
- note removed: "D"
- note removed: "E"
- note removed: "ENTER"
- note removed: "ESC\n"
- note removed: "F"
- note removed: "FN"
- note removed: "G"
- note removed: "H"
- note removed: "I"
- note removed: "J"
- note removed: "K"
- note removed: "L"
- note removed: "LALT"
- note removed: "LCTRL"
- note removed: "LGUI"
- note removed: "LSHIFT"
- note removed: "M"
- note removed: "N"
- note removed: "O"
- note removed: "P"
- note removed: "Q"
- note removed: "R"
- note removed: "RALT"
- note removed: "RCTRL"
- note removed: "RSHIFT"
- note removed: "RTEXT"
- note removed: "S"
- note removed: "SPACE"
- note removed: "T"
- note removed: "TAB"
- note removed: "U"
- note removed: "V"
- note removed: "W"
- note removed: "X"
- note removed: "Y"
- note removed: "Z"
- note removed: "["
- note removed: "\"
- note removed: "]"
- note removed: "backspace"
