File: matrix.sch (KiCad schematic (older format))
At the start: 143 parts

Commit message: default GH60 Keyboard
Parts:
- added DC1, DC2: LED, mx1a:MX1A-led_no3d, symbol LED
- added DC3: LED, symbol LED
- added R4: 300, symbol R
- added S031, S661, S681, S682, S691, S692: MX1A, mx1a:MX1A_no3d, symbol MX1A
- D01: renamed from D4; symbol device:DIODE -> DIODE
- D02: renamed from D5; symbol device:DIODE -> DIODE
- D03: renamed from D6; symbol device:DIODE -> DIODE
- D04: renamed from D7; symbol device:DIODE -> DIODE
- D05: renamed from D8; symbol device:DIODE -> DIODE
- D06: renamed from D9; symbol device:DIODE -> DIODE
- D07: renamed from D10; symbol device:DIODE -> DIODE
- D08: renamed from D11; symbol device:DIODE -> DIODE
- D09: renamed from D12; symbol device:DIODE -> DIODE
- D10: renamed from D13; symbol device:DIODE -> DIODE
- D11: renamed from D14; symbol device:DIODE -> DIODE
- D12: renamed from D15; symbol device:DIODE -> DIODE
- D13: renamed from D16; symbol device:DIODE -> DIODE
- D14: renamed from D17; symbol device:DIODE -> DIODE
- D15: renamed from D18; symbol device:DIODE -> DIODE
- D16: renamed from D19; symbol device:DIODE -> DIODE
- D17: renamed from D20; symbol device:DIODE -> DIODE
- D18: renamed from D21; symbol device:DIODE -> DIODE
- D19: renamed from D22; symbol device:DIODE -> DIODE
- D21: renamed from D23; symbol device:DIODE -> DIODE
- D22: renamed from D24; symbol device:DIODE -> DIODE
- D23: renamed from D25; symbol device:DIODE -> DIODE
- D24: renamed from D26; symbol device:DIODE -> DIODE
- D26: renamed from D27; symbol device:DIODE -> DIODE
- D27: renamed from D28; symbol device:DIODE -> DIODE
- D28: renamed from D29; symbol device:DIODE -> DIODE
- D29: renamed from D30; symbol device:DIODE -> DIODE
- D30: renamed from D31; symbol device:DIODE -> DIODE
- D31: renamed from D32; symbol device:DIODE -> DIODE
- D32: renamed from D33; symbol device:DIODE -> DIODE
- D33: renamed from D34; symbol device:DIODE -> DIODE
- D34: renamed from D35; symbol device:DIODE -> DIODE
- D36, D37, D38, D39: symbol device:DIODE -> DIODE
- D41: renamed from D40; symbol device:DIODE -> DIODE
- D42: renamed from D41; symbol device:DIODE -> DIODE
- D43: renamed from D42; symbol device:DIODE -> DIODE
- D44: renamed from D43; symbol device:DIODE -> DIODE
- D46: renamed from D44; symbol device:DIODE -> DIODE
- D47: renamed from D45; symbol device:DIODE -> DIODE
- D48: renamed from D46; symbol device:DIODE -> DIODE
- D49: renamed from D47; symbol device:DIODE -> DIODE
- D50: renamed from D48; symbol device:DIODE -> DIODE
- D51: renamed from D49; symbol device:DIODE -> DIODE
- D52: renamed from D50; symbol device:DIODE -> DIODE
- D53: renamed from D51; symbol device:DIODE -> DIODE
- D54: renamed from D52; symbol device:DIODE -> DIODE
- D55: renamed from D53; symbol device:DIODE -> DIODE
- D56: renamed from D54; symbol device:DIODE -> DIODE
- D57: renamed from D55; symbol device:DIODE -> DIODE
- D58: renamed from D56; symbol device:DIODE -> DIODE
- D59: renamed from D57; symbol device:DIODE -> DIODE
- D60: renamed from D58; symbol device:DIODE -> DIODE
- D61: renamed from D59; symbol device:DIODE -> DIODE
- D62: renamed from D60; symbol device:DIODE -> DIODE
- D63: renamed from D61; symbol device:DIODE -> DIODE
- D64: renamed from D62; symbol device:DIODE -> DIODE
- D65: renamed from D63; symbol device:DIODE -> DIODE
- D66: renamed from D64; symbol device:DIODE -> DIODE
- D67: renamed from D65; symbol device:DIODE -> DIODE
- D68: renamed from D66; symbol device:DIODE -> DIODE
- D69: renamed from D67; symbol device:DIODE -> DIODE
- D70: renamed from D68; symbol device:DIODE -> DIODE
- S01: renamed from S3; footprint keyswitches:MX -> mx1a:MX1A; symbol mx1a-simple:MX1A -> MX1A
- S02: renamed from S4; footprint keyswitches:MX -> mx1a:MX1A; symbol mx1a-simple:MX1A -> MX1A
- S03: renamed from S5; footprint keyswitches:MX -> mx1a:MX1A; symbol mx1a-simple:MX1A -> MX1A
- S04: renamed from S6; footprint keyswitches:MX -> mx1a:MX1A; symbol mx1a-simple:MX1A -> MX1A
- S041: renamed from S7; footprint keyswitches:MX -> mx1a:MX1A_no3d; symbol mx1a-simple:MX1A -> MX1A
- S05: renamed from S8; footprint keyswitches:MX -> mx1a:MX1A; symbol mx1a-simple:MX1A -> MX1A
- S0512: renamed from S2; footprint keyswitches:MX -> mx1a:MX1A_no3d; symbol mx1a-simple:MX1A -> MX1A
- S06: renamed from S9; footprint keyswitches:MX -> mx1a:MX1A; symbol mx1a-simple:MX1A -> MX1A
- S07: renamed from S10; footprint keyswitches:MX -> mx1a:MX1A; symbol mx1a-simple:MX1A -> MX1A
- S08: renamed from S11; footprint keyswitches:MX -> mx1a:MX1A; symbol mx1a-simple:MX1A -> MX1A
- S09: renamed from S12; footprint keyswitches:MX -> mx1a:MX1A_no3d; symbol mx1a-simple:MX1A -> MX1A
- S10: renamed from S13; footprint keyswitches:MX -> mx1a:MX1A; symbol mx1a-simple:MX1A -> MX1A
- S101: renamed from S15; footprint keyswitches:MX -> mx1a:MX1A_no3d; symbol mx1a-simple:MX1A -> MX1A
- S102: renamed from S14; footprint keyswitches:MX -> mx1a:MX1A_no3d; symbol mx1a-simple:MX1A -> MX1A
- S11: renamed from S17; footprint keyswitches:MX -> mx1a:MX1A; symbol mx1a-simple:MX1A -> MX1A
- S12: renamed from S18; footprint keyswitches:MX -> mx1a:MX1A; symbol mx1a-simple:MX1A -> MX1A
- S13: renamed from S19; footprint keyswitches:MX -> mx1a:MX1A; symbol mx1a-simple:MX1A -> MX1A
- S14: renamed from S20; footprint keyswitches:MX -> mx1a:MX1A; symbol mx1a-simple:MX1A -> MX1A
- S15: renamed from S21; footprint keyswitches:MX -> mx1a:MX1A; symbol mx1a-simple:MX1A -> MX1A
- S151: renamed from S16; footprint keyswitches:MX -> mx1a:MX1A_no3d; symbol mx1a-simple:MX1A -> MX1A
- S16: renamed from S22; footprint keyswitches:MX -> mx1a:MX1A; symbol mx1a-simple:MX1A -> MX1A
- S17: renamed from S23; footprint keyswitches:MX -> mx1a:MX1A; symbol mx1a-simple:MX1A -> MX1A
- S18: renamed from S24; footprint keyswitches:MX -> mx1a:MX1A; symbol mx1a-simple:MX1A -> MX1A
- S19: renamed from S25; footprint keyswitches:MX -> mx1a:MX1A; symbol mx1a-simple:MX1A -> MX1A
- S21: renamed from S26; footprint keyswitches:MX -> mx1a:MX1A; symbol mx1a-simple:MX1A -> MX1A
- S22: renamed from S27; footprint keyswitches:MX -> mx1a:MX1A; symbol mx1a-simple:MX1A -> MX1A
- S23: renamed from S28; footprint keyswitches:MX -> mx1a:MX1A; symbol mx1a-simple:MX1A -> MX1A
- S24: renamed from S29; footprint keyswitches:MX -> mx1a:MX1A; symbol mx1a-simple:MX1A -> MX1A
- S26: renamed from S31; footprint keyswitches:MX -> mx1a:MX1A; symbol mx1a-simple:MX1A -> MX1A
- S27: renamed from S32; footprint keyswitches:MX -> mx1a:MX1A; symbol mx1a-simple:MX1A -> MX1A
- S28: renamed from S33; footprint keyswitches:MX -> mx1a:MX1A; symbol mx1a-simple:MX1A -> MX1A
- S29: renamed from S34; footprint keyswitches:MX -> mx1a:MX1A; symbol mx1a-simple:MX1A -> MX1A
- S30: footprint keyswitches:MX -> mx1a:MX1A; symbol mx1a-simple:MX1A -> MX1A
- S301: renamed from S36; footprint keyswitches:MX -> mx1a:MX1A_no3d; symbol mx1a-simple:MX1A -> MX1A
- S302: renamed from S35; footprint keyswitches:MX -> mx1a:MX1A_no3d; symbol mx1a-simple:MX1A -> MX1A
- S31: renamed from S37; footprint keyswitches:MX -> mx1a:MX1A; symbol mx1a-simple:MX1A -> MX1A
- S32: renamed from S38; footprint keyswitches:MX -> mx1a:MX1A; symbol mx1a-simple:MX1A -> MX1A
- S33: renamed from S39; footprint keyswitches:MX -> mx1a:MX1A; symbol mx1a-simple:MX1A -> MX1A
- S34: renamed from S40; footprint keyswitches:MX -> mx1a:MX1A; symbol mx1a-simple:MX1A -> MX1A
- S36: renamed from S41; footprint keyswitches:MX -> mx1a:MX1A; symbol mx1a-simple:MX1A -> MX1A
- S37: renamed from S42; footprint keyswitches:MX -> mx1a:MX1A; symbol mx1a-simple:MX1A -> MX1A
- S38: renamed from S43; footprint keyswitches:MX -> mx1a:MX1A; symbol mx1a-simple:MX1A -> MX1A
- S39: renamed from S44; footprint keyswitches:MX -> mx1a:MX1A; symbol mx1a-simple:MX1A -> MX1A
- S41: renamed from S45; footprint keyswitches:MX -> mx1a:MX1A; symbol mx1a-simple:MX1A -> MX1A
- S42: renamed from S46; footprint keyswitches:MX -> mx1a:MX1A; symbol mx1a-simple:MX1A -> MX1A
- S43: renamed from S47; footprint keyswitches:MX -> mx1a:MX1A; symbol mx1a-simple:MX1A -> MX1A
- S44: renamed from S48; footprint keyswitches:MX -> mx1a:MX1A; symbol mx1a-simple:MX1A -> MX1A
- S46: renamed from S49; footprint keyswitches:MX -> mx1a:MX1A; symbol mx1a-simple:MX1A -> MX1A
- S47: renamed from S50; footprint keyswitches:MX -> mx1a:MX1A; symbol mx1a-simple:MX1A -> MX1A
- S48: renamed from S51; footprint keyswitches:MX -> mx1a:MX1A; symbol mx1a-simple:MX1A -> MX1A
- S49: renamed from S52; footprint keyswitches:MX -> mx1a:MX1A; symbol mx1a-simple:MX1A -> MX1A
- S50: renamed from S53; footprint keyswitches:MX -> mx1a:MX1A_no3d; symbol mx1a-simple:MX1A -> MX1A
- S51: renamed from S55; footprint keyswitches:MX -> mx1a:MX1A; symbol mx1a-simple:MX1A -> MX1A
- S52: renamed from S56; footprint keyswitches:MX -> mx1a:MX1A; symbol mx1a-simple:MX1A -> MX1A
- S53: renamed from S57; footprint keyswitches:MX -> mx1a:MX1A; symbol mx1a-simple:MX1A -> MX1A
- S54: renamed from S58; footprint keyswitches:MX -> mx1a:MX1A; symbol mx1a-simple:MX1A -> MX1A
- S55: renamed from S59; footprint keyswitches:MX -> mx1a:MX1A; symbol mx1a-simple:MX1A -> MX1A
- S552: renamed from S54; footprint keyswitches:MX -> mx1a:MX1A_no3d; symbol mx1a-simple:MX1A -> MX1A
- S56: renamed from S60; footprint keyswitches:MX -> mx1a:MX1A; symbol mx1a-simple:MX1A -> MX1A
- S57: renamed from S61; footprint keyswitches:MX -> mx1a:MX1A; symbol mx1a-simple:MX1A -> MX1A
- S58: renamed from S62; footprint keyswitches:MX -> mx1a:MX1A; symbol mx1a-simple:MX1A -> MX1A
- S59: renamed from S63; footprint keyswitches:MX -> mx1a:MX1A; symbol mx1a-simple:MX1A -> MX1A
- S60: renamed from S64; footprint keyswitches:MX -> mx1a:MX1A; symbol mx1a-simple:MX1A -> MX1A
- S601: renamed from S65; footprint keyswitches:MX -> mx1a:MX1A_no3d; symbol mx1a-simple:MX1A -> MX1A
- S602: renamed from S66; footprint keyswitches:MX -> mx1a:MX1A_no3d; symbol mx1a-simple:MX1A -> MX1A
- S61: renamed from S68; footprint keyswitches:MX -> mx1a:MX1A; symbol mx1a-simple:MX1A -> MX1A
- S62: renamed from S69; footprint keyswitches:MX -> mx1a:MX1A; symbol mx1a-simple:MX1A -> MX1A
- S63: renamed from S70; footprint keyswitches:MX -> mx1a:MX1A_no3d; symbol mx1a-simple:MX1A -> MX1A
- S64: renamed from S71; footprint keyswitches:MX -> mx1a:MX1A_no3d; symbol mx1a-simple:MX1A -> MX1A
- S641: renamed from S72; footprint keyswitches:MX -> mx1a:MX1A_no3d; symbol mx1a-simple:MX1A -> MX1A
- S65: renamed from S67; footprint keyswitches:MX -> mx1a:MX1A; symbol mx1a-simple:MX1A -> MX1A
- S6512: renamed from S73; footprint keyswitches:MX -> mx1a:MX1A_no3d; symbol mx1a-simple:MX1A -> MX1A
- S66: renamed from S77; footprint keyswitches:MX -> mx1a:MX1A; symbol mx1a-simple:MX1A -> MX1A
- S67: renamed from S79; footprint keyswitches:MX -> mx1a:MX1A; symbol mx1a-simple:MX1A -> MX1A
- S68: renamed from S80; footprint keyswitches:MX -> mx1a:MX1A; symbol mx1a-simple:MX1A -> MX1A
- S69: renamed from S82; footprint keyswitches:MX -> mx1a:MX1A; symbol mx1a-simple:MX1A -> MX1A
- S70: renamed from S76; footprint keyswitches:MX -> mx1a:MX1A; symbol mx1a-simple:MX1A -> MX1A
- S7012: renamed from S84; footprint keyswitches:MX -> mx1a:MX1A_no3d; symbol mx1a-simple:MX1A -> MX1A
Connections:
- net labels added: CAPS_LED, VCC
- wire segments 394 -> 254
